Commit message: updated joint position and velocity limits

File: fanuc_m800ia_support/urdf/m800ia60_macro.xacro (robot description, xacro)
@@ -115,5 +115,5 @@
       <child link="${prefix}link_1"/>
       <axis xyz="0 0 1"/>
-      <limit lower="${radians(-185)}" upper="${radians(185)}" effort="0" velocity="${radians(105)}"/>
+      <limit lower="${radians(-185)}" upper="${radians(185)}" effort="0" velocity="${radians(150)}"/>
     </joint>
     <joint name="${prefix}joint_2" type="revolute">
@@ -122,5 +122,5 @@
       <child link="${prefix}link_2"/>
       <axis xyz="0 1 0"/>
-      <limit lower="${radians(-60)}" upper="${radians(76)}" effort="0" velocity="${radians(90)}"/>
+      <limit lower="${radians(-90)}" upper="${radians(135)}" effort="0" velocity="${radians(150)}"/>
     </joint>
     <joint name="${prefix}joint_3" type="revolute">
@@ -129,5 +129,5 @@
       <child link="${prefix}link_3"/>
       <axis xyz="0 -1 0"/>
-      <limit lower="${radians(-121)}" upper="${radians(180)}" effort="0" velocity="${radians(85)}"/>
+      <limit lower="${radians(-160)}" upper="${radians(180)}" effort="0" velocity="${radians(150)}"/>
     </joint>
     <joint name="${prefix}joint_4" type="revolute">
@@ -136,5 +136,5 @@
       <child link="${prefix}link_4"/>
       <axis xyz="-1 0 0"/>
-      <limit lower="${radians(-360)}" upper="${radians(360)}" effort="0" velocity="${radians(120)}"/>
+      <limit lower="${radians(-360)}" upper="${radians(360)}" effort="0" velocity="${radians(260)}"/>
     </joint>
     <joint name="${prefix}joint_5" type="revolute">
@@ -143,5 +143,5 @@
       <child link="${prefix}link_5"/>
       <axis xyz="0 -1 0"/>
-      <limit lower="${radians(-125)}" upper="${radians(125)}" effort="0" velocity="${radians(120)}"/>
+      <limit lower="${radians(-125)}" upper="${radians(125)}" effort="0" velocity="${radians(260)}"/>
     </joint>
     <joint name="${prefix}joint_6" type="revolute">
@@ -150,5 +150,5 @@
       <child link="${prefix}link_6"/>
       <axis xyz="-1 0 0"/>
-      <limit lower="${radians(-360)}" upper="${radians(360)}" effort="0" velocity="${radians(200)}"/>
+      <limit lower="${radians(-360)}" upper="${radians(360)}" effort="0" velocity="${radians(400)}"/>
     </joint>
     <!-- ROS-Industrial 'base' frame: base_link to Fanuc World Coordinates transform -->
